File: hardware/LBD.kicad_sch (KiCad schematic)
At the start: 18 parts, among them U1 RP2040, Y1 Crystal_GND24

Commit message: swd
Parts:
- added J1: Conn_01x03_Pin, symbol Connector:Conn_01x03_Pin
- Y1: value Crystal_GND24 -> 12 MHz
Connections:
- net GND: now also J1.2 (Pin_2)
- new net SWCLK: J1.3 (Pin_3)
- new net SWDIO: J1.1 (Pin_1)
Other:
- moved on the sheet: C12, C13, C17, C18, C19, C20
