File: hardware/LBD.kicad_sch (KiCad schematic)
At the start: 14 parts, among them J1 Conn_01x03_Pin, U1 RP2040, Y1 12 MHz

Commit message: refactor: update display value from LED to IN-S126ESGHIR
Parts:
- D1, D2, D3, D4, D5, D6, D7: value LED -> IN-S126ESGHIR
Changed lines of the file:
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@@
 			)
 		)
-		(property "Value" "LED"
+		(property "Value" "IN-S126ESGHIR"
 			(at 202.8825 123.19 0)
 			(show_name no)
@@
 			)
 		)
-		(property "Value" "LED"
+		(property "Value" "IN-S126ESGHIR"
 			(at 220.6625 107.95 0)
 			(show_name no)
@@
 			)
 		)
-		(property "Value" "LED"
+		(property "Value" "IN-S126ESGHIR"
 			(at 202.8825 111.76 0)
 			(show_name no)
@@
 			)
 		)
-		(property "Value" "LED"
+		(property "Value" "IN-S126ESGHIR"
 			(at 240.9825 116.84 0)
 			(show_name no)
@@
 			)
 		)
-		(property "Value" "LED"
+		(property "Value" "IN-S126ESGHIR"
 			(at 201.6125 99.06 0)
 			(show_name no)
@@
 			)
 		)
-		(property "Value" "LED"
+		(property "Value" "IN-S126ESGHIR"
 			(at 220.6625 97.79 0)
 			(show_name no)
@@
 			)
 		)
-		(property "Value" "LED"
+		(property "Value" "IN-S126ESGHIR"
 			(at 221.9325 125.73 0)
 			(show_name no)

Commit message: feat: implement IR matrix
Parts:
- removed D1, D2, D3, D4, D5, D6, D7: IN-S126ESGHIR, LBD_Footprints:LED_IN-S12_INL, symbol Device:LED
Connections:
- net Infared/IR_GATE: now reaches U1.4 (GPIO2)
Other:
- added sheet Infared (infared.kicad_sch)
- moved on the sheet: C4, C5, J1, R6, R9, U1, Y1
