File: hardware/LBD.kicad_sch (KiCad schematic)
At the start: 7 parts, among them J1 Conn_01x03_Pin, U1 RP2040, Y1 12 MHz

Commit message: style: drop farad suffix from capacitor values
Parts:
- C4, C5: value 15pF -> 15p
Changed lines of the file:
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@@
 			)
 		)
-		(property "Value" "15pF"
+		(property "Value" "15p"
 			(at 48.2663 120.65 90)
 			(show_name no)
@@
 			)
 		)
-		(property "Value" "15pF"
+		(property "Value" "15p"
 			(at 48.2663 110.49 90)
 			(show_name no)

Commit message: feat: assign footprints for resistors and caps
Parts:
- C4, C5: footprint (none) -> Capacitor_SMD:C_0201_0603Metric
- R6: footprint (none) -> Resistor_SMD:R_0603_1608Metric
- R9: footprint (none) -> Resistor_SMD:R_0201_0603Metric
Changed lines of the file:
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@@
 			)
 		)
-		(property "Footprint" ""
+		(property "Footprint" "Resistor_SMD:R_0603_1608Metric"
 			(at 83.566 125.476 90)
 			(hide yes)
@@
 			)
 		)
-		(property "Footprint" ""
+		(property "Footprint" "Capacitor_SMD:C_0201_0603Metric"
 			(at 48.26 124.46 0)
 			(hide yes)
@@
 			)
 		)
-		(property "Footprint" ""
+		(property "Footprint" "Capacitor_SMD:C_0201_0603Metric"
 			(at 48.26 114.3 0)
 			(hide yes)
@@
 			)
 		)
-		(property "Footprint" ""
+		(property "Footprint" "Resistor_SMD:R_0201_0603Metric"
 			(at 72.644 67.056 90)
 			(hide yes)

Commit message: feat: add footprints for button and pin header
Parts:
- J1: footprint (none) -> Connector_PinHeader_2.54mm:PinHeader_1x03_P2.54mm_Vertical_SMD_Pin1Left
Changed lines of the file:
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@@
 			)
 		)
-		(property "Footprint" ""
+		(property "Footprint" "Connector_PinHeader_2.54mm:PinHeader_1x03_P2.54mm_Vertical_SMD_Pin1Left"
 			(at 36.83 161.29 0)
 			(hide yes)

Commit message: feat: assign missing footprints
Parts:
- Y1: footprint (none) -> Crystal:Crystal_SMD_3225-4Pin_3.2x2.5mm
Changed lines of the file:
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@@
 			)
 		)
-		(property "Footprint" ""
+		(property "Footprint" "Crystal:Crystal_SMD_3225-4Pin_3.2x2.5mm"
 			(at 58.42 119.38 0)
 			(hide yes)
