File: hardware/flash.kicad_sch (KiCad schematic)
At the start: 5 parts, among them SW2 SW_Push, U5 W25Q128JVSIQ

Commit message: added bom generator
Parts:
- SW2: value SW_Push -> BOOTSEL
Changed lines of the file:
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@@
 			)
 		)
-		(property "Value" "SW_Push"
+		(property "Value" "BOOTSEL"
 			(at 102.87 92.71 0)
 			(show_name no)

Commit message: docs(sheet): update title of schematic sheets
Other:
- company: (none) -> Chaos
- title: (none) -> LBD (Lott-Bespitting Diode)
Changed lines of the file:
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@@
 	(generator_version "10.0")
 	(paper "A4")
+	(title_block
+		(title "LBD (Lott-Bespitting Diode)")
+		(date "2026-06-27")
+		(rev "v1.0")
+		(company "Chaos")
+	)
 	(junction
 		(at 129.54 97.79)
