File: hardware/flash.kicad_sch (KiCad schematic)
At the start: 5 parts, among them SW2 BOOTSEL, U5 W25Q128JVSIQ

Commit message: style: drop farad suffix from capacitor values
Parts:
- C16: value 100nF -> 100n
Changed lines of the file:
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@@
 			)
 		)
-		(property "Value" "100nF"
+		(property "Value" "100n"
 			(at 198.12 97.7962 0)
 			(show_name no)

Commit message: feat: assign footprints for resistors and caps
Parts:
- C16: footprint (none) -> Capacitor_SMD:C_0201_0603Metric
- R7, R8: footprint (none) -> Resistor_SMD:R_0201_0603Metric
Changed lines of the file:
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@@
 			)
 		)
-		(property "Footprint" ""
+		(property "Footprint" "Resistor_SMD:R_0201_0603Metric"
 			(at 114.046 98.806 90)
 			(hide yes)
@@
 			)
 		)
-		(property "Footprint" ""
+		(property "Footprint" "Capacitor_SMD:C_0201_0603Metric"
 			(at 195.58 96.52 0)
 			(hide yes)
@@
 			)
 		)
-		(property "Footprint" ""
+		(property "Footprint" "Resistor_SMD:R_0201_0603Metric"
 			(at 128.524 87.376 90)
 			(hide yes)

Commit message: feat: add footprints for button and pin header
Parts:
- SW2: footprint (none) -> Button_Switch_SMD:SW_SPST_B3U-1000P
Changed lines of the file:
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@@
 			)
 		)
-		(property "Footprint" ""
+		(property "Footprint" "Button_Switch_SMD:SW_SPST_B3U-1000P"
 			(at 102.87 92.71 0)
 			(hide yes)

Commit message: feat: assign missing footprints
Parts:
- U5: footprint W25Q128JVSIQ:SOIC127P790X216-8N -> LBD_Footprints:W25Q128JVSIQ
Changed lines of the file:
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@@
 			)
 		)
-		(property "Footprint" "W25Q128JVSIQ:SOIC127P790X216-8N"
+		(property "Footprint" "LBD_Footprints:W25Q128JVSIQ"
 			(at 158.75 105.41 0)
 			(hide yes)
