File: hardware/infared.kicad_sch (KiCad schematic)
At the start: 17 parts, among them Q1 AO3400A

Commit message: docs(sheet): update title of schematic sheets
Other:
- company: (none) -> Chaos
- title: (none) -> LBD (Lott-Bespitting Diode)
Changed lines of the file:
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@@
 	(generator_version "10.0")
 	(paper "A4")
+	(title_block
+		(title "LBD (Lott-Bespitting Diode)")
+		(date "2026-06-27")
+		(rev "v1.0")
+		(company "Chaos")
+	)
 	(junction
 		(at 99.06 68.58)
