File: hardware/power.kicad_sch (KiCad schematic)
At the start: 16 parts, among them U4 TPSM828214SILR

Commit message: docs(sheet): update title of schematic sheets
Other:
- company: (none) -> Chaos
- title: (none) -> LBD (Lott-Bespitting Diode)
Changed lines of the file:
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@@
 	(generator_version "10.0")
 	(paper "A4")
+	(title_block
+		(title "LBD (Lott-Bespitting Diode)")
+		(date "2026-06-27")
+		(rev "v1.0")
+		(company "Chaos")
+	)
 	(rectangle
 		(start 15.24 171.45)
